File: pcb/controler/controler.kicad_sch (KiCad schematic)
At the start: 0 parts

Commit message: added esp32 to schematic
Parts:
- added U1: ESP32-S3-MINI-1, RF_Module:ESP32-S2-MINI-1, symbol RF_Module:ESP32-S3-MINI-1
Connections:
- new net: U1.1 (GND), U1.2 (GND), U1.42 (GND), U1.43 (GND), U1.46 (GND), U1.47 (GND), U1.48 (GND), U1.49 (GND), U1.50 (GND), U1.51 (GND), U1.52 (GND), U1.53 (GND), U1.54 (GND), U1.55 (GND), U1.56 (GND), U1.57 (GND), U1.58 (GND), U1.59 (GND), U1.60 (GND), U1.61 (GND), U1.62 (GND), U1.63 (GND), U1.64 (GND), U1.65 (GND)
Changed lines of the file:
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@@
 	(generator_version "9.0")
 	(paper "A4")
+	(symbol
+		(lib_id "RF_Module:ESP32-S3-MINI-1")
+		(at 143.51 78.74 0)
+		(unit 1)
+		(exclude_from_sim no)
+		(in_bom yes)
+		(on_board yes)
+		(dnp no)
+		(fields_autoplaced yes)
+		(property "Reference" "U1"
+			(at 145.6533 45.72 0)
+			(effects
+				(font
+					(size 1.27 1.27)
+				)
+				(justify left)
+			)
+		)
+		(property "Value" "ESP32-S3-MINI-1"
+			(at 145.6533 48.26 0)
+			(effects
+				(font
+					(size 1.27 1.27)
+				)
+				(justify left)
+			)
+		)
+		(property "Footprint" "RF_Module:ESP32-S2-MINI-1"
+			(at 158.75 107.95 0)
+			(effects
+				(font
+					(size 1.27 1.27)
+				)
+				(hide yes)
+			)
+		)
+		(property "Datasheet" "https://www.espressif.com/sites/default/files/documentation/esp32-s3-mini-1_mini-1u_datasheet_en.pdf"
+			(at 143.51 38.1 0)
+			(effects
+				(font
+					(size 1.27 1.27)
+				)
+				(hide yes)
+			)
+		)
+		(property "Description" "RF Module, ESP32-S3 SoC, Wi-Fi 802.11b/g/n, Bluetooth, BLE, 32-bit, 3.3V, SMD, onboard antenna"
+			(at 143.51 35.56 0)
+			(effects
+				(font
+					(size 1.27 1.27)
+				)
+				(hide yes)
+			)
+		)
+		(pin "41"
+		)
+		(pin "38"
+		)
+		(pin "34"
+		)
+		(pin "21"
+		)
+		(pin "48"
+		)
+		(pin "51"
+		)
+		(pin "11"
+		)
+		(pin "12"
+		)
+		(pin "47"
+		)
+		(pin "44"
+		)
+		(pin "7"
+		)
+		(pin "5"
+		)
+		(pin "20"
+		)
+		(pin "10"
+		)
+		(pin "35"
+		)
+		(pin "17"
+		)
+		(pin "22"
+		)
+		(pin "37"
+		)
+		(pin "49"
+		)
+		(pin "26"
+		)
+		(pin "4"
+		)
+		(pin "30"
+		)
+		(pin "24"
+		)
+		(pin "36"
+		)
+		(pin "8"
+		)
+		(pin "43"
+		)
+		(pin "42"
+		)
+		(pin "2"
+		)
+		(pin "6"
+		)
+		(pin "9"
+		)
+		(pin "50"
+		)
+		(pin "19"
+		)
+		(pin "16"
+		)
+		(pin "45"
+		)
+		(pin "1"
+		)
+		(pin "14"
+		)
+		(pin "55"
+		)
+		(pin "56"
+		)
+		(pin "25"
+		)
+		(pin "53"
+		)
+		(pin "54"
+		)
+		(pin "58"
+		)
+		(pin "3"
+		)
+		(pin "18"
+		)
+		(pin "28"
+		)
+		(pin "59"
+		)
+		(pin "52"
+		)
+		(pin "15"
+		)
+		(pin "13"
+		)
+		(pin "57"
+		)
+		(pin "27"
+		)
+		(pin "29"
+		)
+		(pin "31"
+		)
+		(pin "32"
+		)
+		(pin "23"
+		)
+		(pin "61"
+		)
+		(pin "62"
+		)
+		(pin "63"
+		)
+		(pin "64"
+		)
+		(pin "65"
+		)
+		(pin "39"
+		)
+		(pin "40"
+		)
+		(pin "60"
+		)
+		(pin "33"
+		)
+		(pin "46"
+		)
+		(instances
+			(project ""
+				(path "/21e6d255-55c3-435e-90cd-9955aa11d12c"
+					(reference "U1")
+					(unit 1)
+				)
+			)
+		)
+	)
 	(sheet_instances
 		(path "/"

Commit message: starting controller pcb
Parts:
- removed U1: ESP32-S3-MINI-1, RF_Module:ESP32-S2-MINI-1, symbol RF_Module:ESP32-S3-MINI-1
- added BT1: Battery, symbol Device:Battery
- added C1: 0.33uF, symbol Device:C
- added C2: 0.1uF, symbol Device:C
- added J1: Joystick-1, symbol Connector_Generic:Conn_01x05
- added J2: Joystick-2, symbol Connector_Generic:Conn_01x05
- added J3: OLED Display, symbol Connector_Generic:Conn_01x08
- added SW1: SW_DIP_x01, symbol Switch:SW_DIP_x01
- added U1: ~, symbol controller-library:ESP32-S3-Super-Mini
- added U2: UA78M05QDCYRQ1, Package_TO_SOT_SMD:SOT-223-3_TabPin2, symbol Regulator_Linear:UA78M05QDCYRQ1
- added U3: RFM95W-868S2, RF_Module:HOPERF_RFM9XW_THT, symbol RF_Module:RFM95W-868S2
Connections:
- new net: BT1.1 (+), C1.1, U2.1 (IN)
- new net: C2.1, SW1.1, U2.3 (OUT)
- new net +3.3V: U1.16 (3v3), U3.13 (3.3V)
- new net +5V: J1.2 (Pin_2), J2.2 (Pin_2), J3.2 (Pin_2), SW1.2, U1.18 (5v)
- new net GND: BT1.2 (-), C1.2, C2.2, J1.1 (Pin_1), J2.1 (Pin_1), J3.1 (Pin_1), U1.17 (GND), U2.2 (GND)
