File: pcb/controller/controler.kicad_sch (KiCad schematic)
At the start: 10 parts, among them J1 Joystick-1, J2 Joystick-2, J3 OLED Display, SW1 SW_DIP_x01, U2 UA78M05QDCYRQ1, U3 RFM95W-868S2

Commit message: working on pcb
Connections:
- net GND: no longer U3.1 (GND), U3.10 (GND), U3.8 (GND)
- net A0: no longer names the net of J1.3 (Pin_3)
- net A1: no longer names the net of J1.4 (Pin_4)
- net A2: no longer names the net of J2.3 (Pin_3)
- net A3: no longer names the net of J2.4 (Pin_4)
- net CS_1: no longer names the net of U3.5 (NSS)
- net CS_2: no longer names the net of U1.10 (GP8)
- net CS_2: no longer J3.4 (Pin_4)
- net MISO: no longer names the net of U3.2 (MISO)
- net MOSI: no longer names the net of J3.8 (Pin_8)
- net MOSI: no longer U3.3 (MOSI)
- net OLED_DC: no longer names the net of J3.6 (Pin_6)
- net OLED_RST: no longer names the net of J3.5 (Pin_5)
- net SCK: no longer names the net of J3.7 (Pin_7)
- net SCK: no longer U3.4 (SCK)
